File: plonck.sch (KiCad schematic (older format))
At the start: 127 parts, among them J1 Battery_connector, J2 SWD, Q1 Q_PMOS_DSG, U1 SRV05-4, U2 MCP73831-2-OT, U3 XC6206PxxxMR-Regulator_Linear, U4 nRF52840_holyiot_18010, q1 USB4085-GF-A_REVA

Commit message: updated some fooprints and added lcsc part numbers
Parts:
- C1, C2: LCSC (none) -> C140782
- C3: LCSC (none) -> C525329
- C4: LCSC (none) -> C162266
- C5: value 4,7uF -> 4.7uF; LCSC (none) -> C162266
- D1, D10, D11, D12, D13, D14, D15, D16, D17, D18, D19, D2, D20, D21, D22, D23, D24, D25, D26, D27, D28, D29, D3, D30, D31, D32, D33, D34, D35, D36, D37, D38, D39, D4, D40, D41, D42, D43, D44, D45, D46, D47, D48, D5, D6, D7, D8, D9: footprint Diode_SMD:D_0805_2012Metric -> Diode_SMD:D_SOD-123; LCSC (none) -> C402213
- D49: footprint Diode_SMD:D_0603_1608Metric -> Diode_SMD:D_SOD-123; LCSC (none) -> C129191
- F1: footprint Fuse:Fuse_0805_2012Metric -> Fuse:Fuse_0603_1608Metric; LCSC (none) -> C151138
- J1: LCSC (none) -> C225424
- Q1: LCSC (none) -> C10487
- R1, R2: value 5.1k -> 5.1k Ω; Digikey (none) -> RMCF0603JT5K10TR-ND; LCSC (none) -> C150387
- R3: Digikey (none) -> RMCF0603JT470RTR-ND; LCSC (none) -> C491208
- R4: Digikey (none) -> RMCF0603JG10K0TR-ND; LCSC (none) -> C98220
- R5: value 100kΩ -> 100k Ω; Digikey (none) -> RMCF0603JG100KTR-ND; LCSC (none) -> C427284
- R6: value 10kΩ -> 10k Ω; Digikey (none) -> RMCF0603JG10K0TR-ND; LCSC (none) -> C98220
- S1: LCSC (none) -> C221856
- U1: LCSC (none) -> C782797
- U2: LCSC (none) -> C424093

Commit message: updated parts and fixed ground fill
Parts:
- removed D49: B130-E3, Diode_SMD:D_SOD-123, symbol Diode:B130-E3
- added D49: B130LAW-7-F, Diode_SMD:D_SMA, symbol Diode:B130LAW-7-F
Changed lines of the file:
@@
 Connection ~ 7675 5350
-$Comp
-L Diode:B130-E3 D49
-U 1 1 605E3BB9
-P 7675 5500
-F 0 "D49" V 7721 5420 50  0000 R CNN
-F 1 "B130-E3" V 7630 5420 50  0000 R CNN
-F 2 "Diode_SMD:D_SOD-123" H 7675 5325 50  0001 C CNN
-F 3 "http://www.vishay.com/docs/88946/b120.pdf" H 7675 5500 50  0001 C CNN
-F 4 "C129191" H 7675 5500 50  0001 C CNN "LCSC"
-	1    7675 5500
-	0    -1   -1   0
-$EndComp
 $Comp
 L kicad-keyboard-parts:XC6206PxxxMR-Regulator_Linear U3
@@
 	1    0    0    -1
 $EndComp
+$Comp
+L Diode:B130LAW-7-F D49
+U 1 1 60833B5C
+P 7575 5500
+F 0 "D49" V 7621 5320 50  0000 R CNN
+F 1 "B130LAW-7-F" V 7475 5675 50  0000 R CNN
+F 2 "Diode_SMD:D_SMA" H 7575 5200 50  0001 C CNN
+F 3 "https://datasheet.lcsc.com/lcsc/1811061926_Diodes-Incorporated-B130LAW-7-F_C129191.pdf" H 7575 5500 50  0001 C CNN
+	1    7575 5500
+	0    -1   -1   0
+$EndComp
 $EndSCHEMATC

Commit message: fixing up via sizes and ground planes
Other:
- moved on the sheet: H1, H2, H3, H4, H5, H6, R6
Changed lines of the file:
@@
 Text Notes 675  5575 0    50   ~ 0
 Debug connector
-Text GLabel 2050 7050 2    50   Input ~ 0
+Text GLabel 2000 6975 2    50   Input ~ 0
 RESET
 $Comp
 L power:+3.3V #PWR025
 U 1 1 6079A726
-P 1975 7350
-F 0 "#PWR025" H 1975 7200 50  0001 C CNN
-F 1 "+3.3V" H 1990 7523 50  0000 C CNN
-F 2 "" H 1975 7350 50  0001 C CNN
-F 3 "" H 1975 7350 50  0001 C CNN
-	1    1975 7350
+P 1925 7275
+F 0 "#PWR025" H 1925 7125 50  0001 C CNN
+F 1 "+3.3V" H 1940 7448 50  0000 C CNN
+F 2 "" H 1925 7275 50  0001 C CNN
+F 3 "" H 1925 7275 50  0001 C CNN
+	1    1925 7275
 	-1   0    0    1
 $EndComp
@@
 L Device:R_Small R6
 U 1 1 6079D89A
-P 1975 7250
-F 0 "R6" H 2034 7296 50  0000 L CNN
-F 1 "10k Ω" H 2034 7205 50  0000 L CNN
-F 2 "Resistor_SMD:R_0603_1608Metric" H 1975 7250 50  0001 C CNN
-F 3 "~" H 1975 7250 50  0001 C CNN
-F 4 "RMCF0603JG10K0TR-ND" H 1975 7250 50  0001 C CNN "Digikey"
-F 5 "C98220" H 1975 7250 50  0001 C CNN "LCSC"
-	1    1975 7250
-	1    0    0    -1
-$EndComp
-Wire Wire Line
-	1975 7050 1975 7150
+P 1925 7175
+F 0 "R6" H 1984 7221 50  0000 L CNN
+F 1 "10k Ω" H 1984 7130 50  0000 L CNN
+F 2 "Resistor_SMD:R_0603_1608Metric" H 1925 7175 50  0001 C CNN
+F 3 "~" H 1925 7175 50  0001 C CNN
+F 4 "RMCF0603JG10K0TR-ND" H 1925 7175 50  0001 C CNN "Digikey"
+F 5 "C98220" H 1925 7175 50  0001 C CNN "LCSC"
+	1    1925 7175
+	1    0    0    -1
+$EndComp
+Wire Wire Line
+	1925 6975 1925 7075
 $Comp
 L Diode:1N4148W D12
@@
 	1    0    0    -1
 $EndComp
-Connection ~ 1975 7050
-Wire Wire Line
-	1975 7050 2050 7050
+Connection ~ 1925 6975
+Wire Wire Line
+	1925 6975 2000 6975
 $Comp
 L MX_Alps_Hybrid:MX-NoLED MX49
@@
 L Mechanical:MountingHole H2
 U 1 1 60788588
-P 2725 6700
-F 0 "H2" H 2825 6746 50  0000 L CNN
-F 1 "MountingHole" H 2825 6655 50  0000 L CNN
-F 2 "MountingHole:MountingHole_2.7mm_M2.5_Pad_Via" H 2725 6700 50  0001 C CNN
-F 3 "~" H 2725 6700 50  0001 C CNN
-	1    2725 6700
+P 2700 6575
+F 0 "H2" H 2800 6621 50  0000 L CNN
+F 1 "MountingHole" H 2800 6530 50  0000 L CNN
+F 2 "MountingHole:MountingHole_2.7mm_M2.5_Pad_Via" H 2700 6575 50  0001 C CNN
+F 3 "~" H 2700 6575 50  0001 C CNN
+	1    2700 6575
 	1    0    0    -1
 $EndComp
@@
 L Mechanical:MountingHole H3
 U 1 1 6078ED29
-P 2725 6900
-F 0 "H3" H 2825 6946 50  0000 L CNN
-F 1 "MountingHole" H 2825 6855 50  0000 L CNN
-F 2 "MountingHole:MountingHole_2.7mm_M2.5_Pad_Via" H 2725 6900 50  0001 C CNN
-F 3 "~" H 2725 6900 50  0001 C CNN
-	1    2725 6900
+P 2700 6775
+F 0 "H3" H 2800 6821 50  0000 L CNN
+F 1 "MountingHole" H 2800 6730 50  0000 L CNN
+F 2 "MountingHole:MountingHole_2.7mm_M2.5_Pad_Via" H 2700 6775 50  0001 C CNN
+F 3 "~" H 2700 6775 50  0001 C CNN
+	1    2700 6775
 	1    0    0    -1
 $EndComp
@@
 L Mechanical:MountingHole H4
 U 1 1 6078F11A
-P 2725 7100
-F 0 "H4" H 2825 7146 50  0000 L CNN
-F 1 "MountingHole" H 2825 7055 50  0000 L CNN
-F 2 "MountingHole:MountingHole_2.7mm_M2.5_Pad_Via" H 2725 7100 50  0001 C CNN
-F 3 "~" H 2725 7100 50  0001 C CNN
-	1    2725 7100
+P 2700 6975
+F 0 "H4" H 2800 7021 50  0000 L CNN
+F 1 "MountingHole" H 2800 6930 50  0000 L CNN
+F 2 "MountingHole:MountingHole_2.7mm_M2.5_Pad_Via" H 2700 6975 50  0001 C CNN
+F 3 "~" H 2700 6975 50  0001 C CNN
+	1    2700 6975
 	1    0    0    -1
 $EndComp
@@
 L Mechanical:MountingHole H5
 U 1 1 6078F582
-P 2725 7300
-F 0 "H5" H 2825 7346 50  0000 L CNN
-F 1 "MountingHole" H 2825 7255 50  0000 L CNN
-F 2 "MountingHole:MountingHole_2.7mm_M2.5_Pad_Via" H 2725 7300 50  0001 C CNN
-F 3 "~" H 2725 7300 50  0001 C CNN
-	1    2725 7300
+P 2700 7175
+F 0 "H5" H 2800 7221 50  0000 L CNN
+F 1 "MountingHole" H 2800 7130 50  0000 L CNN
+F 2 "MountingHole:MountingHole_2.7mm_M2.5_Pad_Via" H 2700 7175 50  0001 C CNN
+F 3 "~" H 2700 7175 50  0001 C CNN
+	1    2700 7175
 	1    0    0    -1
 $EndComp
@@
 L Mechanical:MountingHole H6
 U 1 1 6078FA1D
-P 2725 7500
-F 0 "H6" H 2825 7546 50  0000 L CNN
-F 1 "MountingHole" H 2825 7455 50  0000 L CNN
-F 2 "MountingHole:MountingHole_2.7mm_M2.5_Pad_Via" H 2725 7500 50  0001 C CNN
-F 3 "~" H 2725 7500 50  0001 C CNN
-	1    2725 7500
+P 2700 7375
+F 0 "H6" H 2800 7421 50  0000 L CNN
+F 1 "MountingHole" H 2800 7330 50  0000 L CNN
+F 2 "MountingHole:MountingHole_2.7mm_M2.5_Pad_Via" H 2700 7375 50  0001 C CNN
+F 3 "~" H 2700 7375 50  0001 C CNN
+	1    2700 7375
 	1    0    0    -1
 $EndComp
@@
 L Mechanical:MountingHole H1
 U 1 1 60786A79
-P 2725 6500
-F 0 "H1" H 2825 6546 50  0000 L CNN
-F 1 "MountingHole" H 2825 6455 50  0000 L CNN
-F 2 "MountingHole:MountingHole_2.7mm_M2.5_Pad_Via" H 2725 6500 50  0001 C CNN
-F 3 "~" H 2725 6500 50  0001 C CNN
-	1    2725 6500
-	1    0    0    -1
-$EndComp
-Wire Notes Line
-	2575 6375 2575 7625
-Wire Notes Line
-	2575 7625 3425 7625
-Wire Notes Line
-	3425 7625 3425 6375
-Wire Notes Line
-	3425 6375 2575 6375
-Text Notes 2575 6350 0    50   ~ 0
+P 2700 6375
+F 0 "H1" H 2800 6421 50  0000 L CNN
+F 1 "MountingHole" H 2800 6330 50  0000 L CNN
+F 2 "MountingHole:MountingHole_2.7mm_M2.5_Pad_Via" H 2700 6375 50  0001 C CNN
+F 3 "~" H 2700 6375 50  0001 C CNN
+	1    2700 6375
+	1    0    0    -1
+$EndComp
+Wire Notes Line
+	2550 7500 3400 7500
+Wire Notes Line
+	3400 7500 3400 6250
+Wire Notes Line
+	3400 6250 2550 6250
+Text Notes 2550 6225 0    50   ~ 0
 Mounting hole
 $Comp
 L PTS525SM15SMTR2LFS:PTS525SM15SMTR2LFS S1
 U 1 1 60794776
-P 1300 7150
-F 0 "S1" H 1300 7517 50  0000 C CNN
-F 1 "PTS525SM15SMTR2LFS" H 1300 7426 50  0000 C CNN
-F 2 "PTS525SM15SMTR2LFS:SW_PTS525SM15SMTR2LFS" H 1300 7150 50  0001 L BNN
-F 3 "" H 1300 7150 50  0001 L BNN
-F 4 "Manufacturer REcommendation" H 1300 7150 50  0001 L BNN "STANDARD"
-F 5 "NA" H 1300 7150 50  0001 L BNN "PARTREV"
-F 6 "C & K" H 1300 7150 50  0001 L BNN "MANUFACTURER"
-F 7 "C221856" H 1300 7150 50  0001 C CNN "LCSC"
-	1    1300 7150
-	1    0    0    -1
-$EndComp
-Wire Wire Line
-	1700 7050 1700 7250
-Wire Wire Line
-	1700 7050 1975 7050
-Connection ~ 1700 7050
+P 1250 7075
+F 0 "S1" H 1250 7442 50  0000 C CNN
+F 1 "PTS525SM15SMTR2LFS" H 1250 7351 50  0000 C CNN
+F 2 "PTS525SM15SMTR2LFS:SW_PTS525SM15SMTR2LFS" H 1250 7075 50  0001 L BNN
+F 3 "" H 1250 7075 50  0001 L BNN
+F 4 "Manufacturer REcommendation" H 1250 7075 50  0001 L BNN "STANDARD"
+F 5 "NA" H 1250 7075 50  0001 L BNN "PARTREV"
+F 6 "C & K" H 1250 7075 50  0001 L BNN "MANUFACTURER"
+F 7 "C221856" H 1250 7075 50  0001 C CNN "LCSC"
+	1    1250 7075
+	1    0    0    -1
+$EndComp
+Wire Wire Line
+	1650 6975 1650 7175
+Wire Wire Line
+	1650 6975 1925 6975
+Connection ~ 1650 6975
 $Comp
 L power:GND #PWR02
 U 1 1 607C6905
-P 900 7250
-F 0 "#PWR02" H 900 7000 50  0001 C CNN
-F 1 "GND" H 905 7077 50  0000 C CNN
-F 2 "" H 900 7250 50  0001 C CNN
-F 3 "" H 900 7250 50  0001 C CNN
-	1    900  7250
-	1    0    0    -1
-$EndComp
-Wire Wire Line
-	900  7050 900  7250
-Connection ~ 900  7250
-Wire Notes Line
-	725  6725 725  7575
-Wire Notes Line
-	725  7575 2375 7575
-Wire Notes Line
-	2375 7575 2375 6725
-Wire Notes Line
-	2375 6725 725  6725
-Text Notes 725  6700 0    50   ~ 0
+P 850 7175
+F 0 "#PWR02" H 850 6925 50  0001 C CNN
+F 1 "GND" H 855 7002 50  0000 C CNN
+F 2 "" H 850 7175 50  0001 C CNN
+F 3 "" H 850 7175 50  0001 C CNN
+	1    850  7175
+	1    0    0    -1
+$EndComp
+Wire Wire Line
+	850  6975 850  7175
+Connection ~ 850  7175
+Wire Notes Line
+	675  6650 675  7500
+Wire Notes Line
+	675  7500 2325 7500
+Wire Notes Line
+	2325 7500 2325 6650
+Wire Notes Line
+	2325 6650 675  6650
+Text Notes 675  6625 0    50   ~ 0
 Reset switch
 $Comp
@@
 	0    -1   -1   0
 $EndComp
+Wire Notes Line
+	2550 6250 2550 7500
 $EndSCHEMATC

Commit message: added missing lcsc part number
Parts:
- C1, C2: value 47 uf -> 47uF; LCSC C140782 -> C19666
- D49: LCSC (none) -> C129191
- F1: value 500mah -> SMD Fuse Fast Blow 500mA; footprint Fuse:Fuse_0603_1608Metric -> Fuse:Fuse_1206_3216Metric; LCSC C151138 -> C163133
- R1, R2: value 5.1k Ω -> 5.1k; LCSC C150387 -> C23186
- R3: value 470 Ω -> 470; LCSC C491208 -> C23179
- R4, R6: value 10k Ω -> 10k; LCSC C98220 -> C25804
- R5: value 100k Ω -> 100k; LCSC C427284 -> C25803
- renumbered C4 to C3, C3 to C4
Changed lines of the file:
@@
 P 8250 1925
 F 0 "R1" V 8250 1925 50  0000 C CNN
-F 1 "5.1k Ω" V 8175 1925 50  0000 C CNN
+F 1 "5.1k" V 8175 1925 50  0000 C CNN
 F 2 "Resistor_SMD:R_0603_1608Metric" H 8250 1925 50  0001 C CNN
 F 3 "~" H 8250 1925 50  0001 C CNN
 F 4 "RMCF0603JT5K10TR-ND" V 8250 1925 50  0001 C CNN "Digikey"
-F 5 "C150387" H 8250 1925 50  0001 C CNN "LCSC"
+F 5 "C23186" H 8250 1925 50  0001 C CNN "LCSC"
 	1    8250 1925
 	0    1    1    0
@@
 P 8250 2025
 F 0 "R2" V 8250 2025 50  0000 C CNN
-F 1 "5.1k Ω" V 8325 2025 50  0000 C CNN
+F 1 "5.1k" V 8325 2025 50  0000 C CNN
 F 2 "Resistor_SMD:R_0603_1608Metric" H 8250 2025 50  0001 C CNN
 F 3 "~" H 8250 2025 50  0001 C CNN
 F 4 "RMCF0603JT5K10TR-ND" V 8250 2025 50  0001 C CNN "Digikey"
-F 5 "C150387" H 8250 2025 50  0001 C CNN "LCSC"
+F 5 "C23186" H 8250 2025 50  0001 C CNN "LCSC"
 	1    8250 2025
 	0    1    1    0
@@
 P 9775 3750
 F 0 "C2" H 9900 3825 50  0000 C CNN
-F 1 "47 uf" H 9950 3700 50  0000 C CNN
+F 1 "47uF" H 9950 3700 50  0000 C CNN
 F 2 "Capacitor_SMD:C_0603_1608Metric" H 9775 3750 50  0001 C CNN
 F 3 "~" H 9775 3750 50  0001 C CNN
-F 4 "C140782" H 9775 3750 50  0001 C CNN "LCSC"
+F 4 "C19666" H 9775 3750 50  0001 C CNN "LCSC"
 	1    9775 3750
 	1    0    0    -1
@@
 $EndComp
 $Comp
-L power:GND #PWR015
+L power:GND #PWR021
 U 1 1 607763AE
 P 1125 5875
-F 0 "#PWR015" H 1125 5625 50  0001 C CNN
+F 0 "#PWR021" H 1125 5625 50  0001 C CNN
 F 1 "GND" V 1130 5747 50  0000 R CNN
 F 2 "" H 1125 5875 50  0001 C CNN
@@
 $EndComp
 $Comp
-L power:+3.3V #PWR017
+L power:+3.3V #PWR023
 U 1 1 607779FE
 P 1125 6275
-F 0 "#PWR017" H 1125 6125 50  0001 C CNN
+F 0 "#PWR023" H 1125 6125 50  0001 C CNN
 F 1 "+3.3V" V 1140 6403 50  0000 L CNN
 F 2 "" H 1125 6275 50  0001 C CNN
@@
 RESET
 $Comp
-L power:+3.3V #PWR025
+L power:+3.3V #PWR028
 U 1 1 6079A726
 P 1925 7275
-F 0 "#PWR025" H 1925 7125 50  0001 C CNN
+F 0 "#PWR028" H 1925 7125 50  0001 C CNN
 F 1 "+3.3V" H 1940 7448 50  0000 C CNN
 F 2 "" H 1925 7275 50  0001 C CNN
@@
 P 1925 7175
 F 0 "R6" H 1984 7221 50  0000 L CNN
-F 1 "10k Ω" H 1984 7130 50  0000 L CNN
+F 1 "10k" H 1984 7130 50  0000 L CNN
 F 2 "Resistor_SMD:R_0603_1608Metric" H 1925 7175 50  0001 C CNN
 F 3 "~" H 1925 7175 50  0001 C CNN
 F 4 "RMCF0603JG10K0TR-ND" H 1925 7175 50  0001 C CNN "Digikey"
-F 5 "C98220" H 1925 7175 50  0001 C CNN "LCSC"
+F 5 "C25804" H 1925 7175 50  0001 C CNN "LCSC"
 	1    1925 7175
 	1    0    0    -1
@@
 P 8100 2225
 F 0 "F1" V 8000 2200 50  0000 C CNN
-F 1 "500mah" V 8200 2250 50  0000 C CNN
-F 2 "Fuse:Fuse_0603_1608Metric" H 8150 2025 50  0001 L CNN
+F 1 "SMD Fuse Fast Blow 500mA" V 8200 2250 50  0000 C CNN
+F 2 "Fuse:Fuse_1206_3216Metric" H 8150 2025 50  0001 L CNN
 F 3 "~" H 8100 2225 50  0001 C CNN
-F 4 "C151138" H 8100 2225 50  0001 C CNN "LCSC"
+F 4 "C163133" H 8100 2225 50  0001 C CNN "LCSC"
 	1    8100 2225
 	0    1    1    0
@@
 P 8775 3075
 F 0 "C1" V 8950 3225 50  0000 C CNN
-F 1 "47 uf" V 8875 3175 50  0000 C CNN
+F 1 "47uF" V 8875 3175 50  0000 C CNN
 F 2 "Capacitor_SMD:C_0603_1608Metric" H 8775 3075 50  0001 C CNN
 F 3 "~" H 8775 3075 50  0001 C CNN
-F 4 "C140782" H 8775 3075 50  0001 C CNN "LCSC"
+F 4 "C19666" H 8775 3075 50  0001 C CNN "LCSC"
 	1    8775 3075
 	0    -1   -1   0
@@
 P 8650 4025
 F 0 "R4" H 8709 4071 50  0000 L CNN
-F 1 "10k Ω" H 8709 3980 50  0000 L CNN
+F 1 "10k" H 8709 3980 50  0000 L CNN
 F 2 "Resistor_SMD:R_0603_1608Metric" H 8650 4025 50  0001 C CNN
 F 3 "~" H 8650 4025 50  0001 C CNN
 F 4 "RMCF0603JG10K0TR-ND" H 8650 4025 50  0001 C CNN "Digikey"
-F 5 "C98220" H 8650 4025 50  0001 C CNN "LCSC"
+F 5 "C25804" H 8650 4025 50  0001 C CNN "LCSC"
 	1    8650 4025
 	1    0    0    -1
@@
 	7575 3700 7775 3700
 $Comp
-L power:VBUS #PWR0107
+L power:VBUS #PWR06
 U 1 1 607C3C76
 P 9050 2975
-F 0 "#PWR0107" H 9050 2825 50  0001 C CNN
+F 0 "#PWR06" H 9050 2825 50  0001 C CNN
 F 1 "VBUS" H 9065 3148 50  0000 C CNN
 F 2 "" H 9050 2975 50  0001 C CNN
@@
 $EndComp
 $Comp
-L power:VBUS #PWR0108
+L power:VBUS #PWR02
 U 1 1 607C53BB
 P 9325 1425
-F 0 "#PWR0108" H 9325 1275 50  0001 C CNN
+F 0 "#PWR02" H 9325 1275 50  0001 C CNN
 F 1 "VBUS" V 9340 1552 50  0000 L CNN
 F 2 "" H 9325 1425 50  0001 C CNN
@@
 $EndComp
 $Comp
-L power:VBUS #PWR0109
+L power:VBUS #PWR05
 U 1 1 607C6C1D
 P 8500 2225
-F 0 "#PWR0109" H 8500 2075 50  0001 C CNN
+F 0 "#PWR05" H 8500 2075 50  0001 C CNN
 F 1 "VBUS" V 8515 2353 50  0000 L CNN
 F 2 "" H 8500 2225 50  0001 C CNN
@@
 	7925 2225 7975 2225
 $Comp
-L power:PWR_FLAG #FLG0102
+L power:PWR_FLAG #FLG02
 U 1 1 607D039D
 P 8400 2225
-F 0 "#FLG0102" H 8400 2300 50  0001 C CNN
+F 0 "#FLG02" H 8400 2300 50  0001 C CNN
 F 1 "PWR_FLAG" H 8400 2398 50  0000 C CNN
 F 2 "" H 8400 2225 50  0001 C CNN
@@
 	8200 2225 8400 2225
 $Comp
-L power:PWR_FLAG #FLG0103
+L power:PWR_FLAG #FLG01
 U 1 1 607D2E30
 P 7975 2225
-F 0 "#FLG0103" H 7975 2300 50  0001 C CNN
+F 0 "#FLG01" H 7975 2300 50  0001 C CNN
 F 1 "PWR_FLAG" H 7975 2398 50  0000 C CNN
 F 2 "" H 7975 2225 50  0001 C CNN
@@
 	3650 4850 3650 7350
 $Comp
-L power:VBUS #PWR0105
+L power:VBUS #PWR026
 U 1 1 607C08D6
 P 5150 6950
-F 0 "#PWR0105" H 5150 6800 50  0001 C CNN
+F 0 "#PWR026" H 5150 6800 50  0001 C CNN
 F 1 "VBUS" H 5165 7123 50  0000 C CNN
 F 2 "" H 5150 6950 50  0001 C CNN
@@
 Row1
 $Comp
-L power:GND #PWR0104
+L power:GND #PWR024
 U 1 1 605A52FF
 P 5550 6450
-F 0 "#PWR0104" H 5550 6200 50  0001 C CNN
+F 0 "#PWR024" H 5550 6200 50  0001 C CNN
 F 1 "GND" V 5555 6322 50  0000 R CNN
 F 2 "" H 5550 6450 50  0001 C CNN
@@
 $EndComp
 $Comp
-L power:GND #PWR0103
+L power:GND #PWR017
 U 1 1 605A4F07
 P 4150 5250
-F 0 "#PWR0103" H 4150 5000 50  0001 C CNN
+F 0 "#PWR017" H 4150 5000 50  0001 C CNN
 F 1 "GND" V 4155 5122 50  0000 R CNN
 F 2 "" H 4150 5250 50  0001 C CNN
@@
 $EndComp
 $Comp
-L power:GND #PWR0102
+L power:GND #PWR018
 U 1 1 605A3997
 P 5550 5250
-F 0 "#PWR0102" H 5550 5000 50  0001 C CNN
+F 0 "#PWR018" H 5550 5000 50  0001 C CNN
 F 1 "GND" V 5555 5122 50  0000 R CNN
 F 2 "" H 5550 5250 50  0001 C CNN
@@
 SWDIO
 $Comp
-L power:+3.3V #PWR0101
+L power:+3.3V #PWR025
 U 1 1 605A080F
 P 4350 6950
-F 0 "#PWR0101" H 4350 6800 50  0001 C CNN
+F 0 "#PWR025" H 4350 6800 50  0001 C CNN
 F 1 "+3.3V" V 4350 7175 50  0000 C CNN
 F 2 "" H 4350 6950 50  0001 C CNN
@@
 	7200 6200 10650 6200
 $Comp
-L power:VBUS #PWR0106
+L power:VBUS #PWR019
 U 1 1 607C2523
 P 7575 5350
-F 0 "#PWR0106" H 7575 5200 50  0001 C CNN
+F 0 "#PWR019" H 7575 5200 50  0001 C CNN
 F 1 "VBUS" V 7590 5477 50  0000 L CNN
 F 2 "" H 7575 5350 50  0001 C CNN
@@
 Connection ~ 8625 5650
 $Comp
-L power:PWR_FLAG #FLG0101
+L power:PWR_FLAG #FLG03
 U 1 1 607EA337
 P 8625 5650
-F 0 "#FLG0101" H 8625 5725 50  0001 C CNN
+F 0 "#FLG03" H 8625 5725 50  0001 C CNN
 F 1 "PWR_FLAG" H 8625 5823 50  0000 C CNN
 F 2 "" H 8625 5650 50  0001 C CNN
@@
 	7200 4650 10650 4650
 $Comp
-L power:GND #PWR014
+L power:GND #PWR015
 U 1 1 6062DC30
 P 7675 4950
-F 0 "#PWR014" H 7675 4700 50  0001 C CNN
+F 0 "#PWR015" H 7675 4700 50  0001 C CNN
 F 1 "GND" H 7680 4777 50  0000 C CNN
 F 2 "" H 7675 4950 50  0001 C CNN
@@
 P 7675 5050
 F 0 "R5" H 7734 5096 50  0000 L CNN
-F 1 "100k Ω" H 7734 5005 50  0000 L CNN
+F 1 "100k" H 7734 5005 50  0000 L CNN
 F 2 "Resistor_SMD:R_0603_1608Metric" H 7675 5050 50  0001 C CNN
 F 3 "~" H 7675 5050 50  0001 C CNN
 F 4 "RMCF0603JG100KTR-ND " H 7675 5050 50  0001 C CNN "Digikey"
-F 5 "C427284" H 7675 5050 50  0001 C CNN "LCSC"
+F 5 "C25803" H 7675 5050 50  0001 C CNN "LCSC"
 	1    7675 5050
 	1    0    0    -1
@@
 	9550 5350 9650 5350
 $Comp
-L Device:C_Small C4
+L Device:C_Small C3
 U 1 1 606134D8
 P 9650 5250
-F 0 "C4" H 9742 5296 50  0000 L CNN
+F 0 "C3" H 9742 5296 50  0000 L CNN
 F 1 "4.7uF" H 9742 5205 50  0000 L CNN
 F 2 "Capacitor_SMD:C_0603_1608Metric" H 9650 5250 50  0001 C CNN
@@
 $EndComp
 $Comp
-L Device:C_Small C3
+L Device:C_Small C4
 U 1 1 6061145D
 P 9975 5250
-F 0 "C3" H 10067 5296 50  0000 L CNN
+F 0 "C4" H 10067 5296 50  0000 L CNN
 F 1 "1uF" H 10067 5205 50  0000 L CNN
 F 2 "Capacitor_SMD:C_0603_1608Metric" H 9975 5250 50  0001 C CNN
@@
 $EndComp
 $Comp
-L power:+3.3V #PWR019
+L power:+3.3V #PWR020
 U 1 1 6060F97E
 P 10225 5350
-F 0 "#PWR019" H 10225 5200 50  0001 C CNN
+F 0 "#PWR020" H 10225 5200 50  0001 C CNN
 F 1 "+3.3V" V 10240 5478 50  0000 L CNN
 F 2 "" H 10225 5350 50  0001 C CNN
@@
 $EndComp
 $Comp
-L power:GND #PWR020
+L power:GND #PWR014
 U 1 1 606067FA
 P 9250 4875
-F 0 "#PWR020" H 9250 4625 50  0001 C CNN
+F 0 "#PWR014" H 9250 4625 50  0001 C CNN
 F 1 "GND" H 9255 4702 50  0000 C CNN
 F 2 "" H 9250 4875 50  0001 C CNN
@@
 $EndComp
 $Comp
-L power:GND #PWR021
+L power:GND #PWR022
 U 1 1 605DA2CB
 P 8075 5950
-F 0 "#PWR021" H 8075 5700 50  0001 C CNN
+F 0 "#PWR022" H 8075 5700 50  0001 C CNN
 F 1 "GND" H 8080 5777 50  0000 C CNN
 F 2 "" H 8075 5950 50  0001 C CNN
@@
 Connection ~ 1650 6975
 $Comp
-L power:GND #PWR02
+L power:GND #PWR027
 U 1 1 607C6905
 P 850 7175
-F 0 "#PWR02" H 850 6925 50  0001 C CNN
+F 0 "#PWR027" H 850 6925 50  0001 C CNN
 F 1 "GND" H 855 7002 50  0000 C CNN
 F 2 "" H 850 7175 50  0001 C CNN
@@
 P 9575 3300
 F 0 "R3" H 9634 3346 50  0000 L CNN
-F 1 "470 Ω" H 9634 3255 50  0000 L CNN
+F 1 "470" H 9634 3255 50  0000 L CNN
 F 2 "Resistor_SMD:R_0603_1608Metric" H 9575 3300 50  0001 C CNN
 F 3 "~" H 9575 3300 50  0001 C CNN
 F 4 "RMCF0603JT470RTR-ND" H 9575 3300 50  0001 C CNN "Digikey"
-F 5 "C491208" H 9575 3300 50  0001 C CNN "LCSC"
+F 5 "C23179" H 9575 3300 50  0001 C CNN "LCSC"
 	1    9575 3300
 	1    0    0    -1
@@
 F 2 "Diode_SMD:D_SMA" H 7575 5200 50  0001 C CNN
 F 3 "https://datasheet.lcsc.com/lcsc/1811061926_Diodes-Incorporated-B130LAW-7-F_C129191.pdf" H 7575 5500 50  0001 C CNN
+F 4 "C129191" H 7575 5500 50  0001 C CNN "LCSC"
 	1    7575 5500
 	0    -1   -1   0

Commit message: bunch of fixes and changes to use only basic parts from lcsc
Parts:
- removed S1: PTS525SM15SMTR2LFS, PTS525SM15SMTR2LFS:SW_PTS525SM15SMTR2LFS, symbol PTS525SM15SMTR2LFS:PTS525SM15SMTR2LFS
- removed U2: MCP73831-2-OT, Package_TO_SOT_SMD:SOT-23-5, symbol Battery_Management:MCP73831-2-OT
- added J3: Reset, Connector_PinHeader_2.00mm:PinHeader_1x02_P2.00mm_Vertical, symbol Connector_Generic:Conn_01x02
- added U2: TP4054-42-SOT25-R, Package_TO_SOT_SMD:TSOT-23-5, symbol Battery_Management:TP4054-42-SOT25-R
- C1, C2: footprint Capacitor_SMD:C_0603_1608Metric -> Capacitor_SMD:C_1206_3216Metric; LCSC C19666 -> C96123
- D49: value B130LAW-7-F -> SS14; symbol Diode:B130LAW-7-F -> Diode:SS14; LCSC C129191 -> C2480
- F1: LCSC C163133 -> (none)
- J1: LCSC C225424 -> (none)
- R6: Digikey RMCF0603JG10K0TR-ND -> (none); LCSC C25804 -> (none)
Connections:
- wire segments 156 -> 154
Other:
- note added: "Reset"
- note removed: "Reset switch"
- moved on the sheet: H1, H2, H3, H4, H5, H6

Commit message: rescue stuff
Parts:
- D49: symbol Diode:SS14 -> plonck-rescue:SS14-Diode
- J1: symbol Connector_Generic:Battery_connector -> plonck-rescue:Battery_connector-Connector_Generic
- J2: symbol Connector_Generic:SWD -> plonck-rescue:SWD-Connector_Generic
- U2: symbol Battery_Management:TP4054-42-SOT25-R -> plonck-rescue:TP4054-42-SOT25-R-Battery_Management
Changed lines of the file:
@@
 ESD protection
 $Comp
-L Connector_Generic:SWD J2
+L plonck-rescue:SWD-Connector_Generic J2
 U 1 1 60775440
 P 1275 5600
@@
 	8900 2475 8900 675
 $Comp
-L Connector_Generic:Battery_connector J1
+L plonck-rescue:Battery_connector-Connector_Generic J1
 U 1 1 605544B8
 P 7875 3450
@@
 $EndComp
 $Comp
-L Diode:SS14 D49
+L plonck-rescue:SS14-Diode D49
 U 1 1 60833B5C
 P 7575 5500
@@
 	675  6425 675  7675
 $Comp
-L Battery_Management:TP4054-42-SOT25-R U2
+L plonck-rescue:TP4054-42-SOT25-R-Battery_Management U2
 U 1 1 608A020D
 P 9050 3625
