File: plonck.sch (KiCad schematic (older format))
At the start: 127 parts, among them J1 Battery_connector, J2 SWD, J3 Reset, Q1 Q_PMOS_DSG, U1 SRV05-4, U2 TP4054-42-SOT25-R, U3 XC6206PxxxMR-Regulator_Linear, U4 nRF52840_holyiot_18010, q1 USB4085-GF-A_REVA

Commit message: various fixes and additions
changed switch footprints to be alps compatible
added descriptive text to bottom row
fixed mounting holes not being connected to ground
fixed incorrectly wired esd chip
added reset switch in default planck position
changed mx3 to normal rotation
changed board outline to move usb port further out
Parts:
- removed J3: Reset, Connector_PinHeader_2.00mm:PinHeader_1x02_P2.00mm_Vertical, symbol Connector_Generic:Conn_01x02
- added SW1: SW_Push, Button_Switch_SMD:SW_Push_SPST_NO_Alps_SKRK, symbol Switch:SW_Push
- H1, H2, H3, H4, H5, H6: symbol Mechanical:MountingHole -> Mechanical:MountingHole_Pad
- MX1, MX10, MX11, MX12, MX13, MX14, MX15, MX16, MX17, MX18, MX19, MX2, MX20, MX21, MX22, MX23, MX24, MX25, MX26, MX27, MX28, MX29, MX3, MX30, MX31, MX32, MX33, MX34, MX35, MX36, MX37, MX38, MX39, MX4, MX40, MX41, MX42, MX43, MX44, MX45, MX46, MX47, MX48, MX5, MX6, MX7, MX8, MX9: footprint MX_Only:MXOnly-1U-NoLED -> MX_Alps_Hybrid:MX-1U-NoLED
- MX49, MX50, MX51: footprint MX_Only:MXOnly-2U-ReversedStabilizers-NoLED -> MX_Alps_Hybrid:MX-2U-ReversedStabilizers-NoLED
Connections:
- net D+: now also U1.6 (IO4); no longer U1.3 (IO2)
- net D-: now also U1.1 (IO1); no longer U1.4 (IO3)
- net GND: now also H1.1, H2.1, H3.1, H4.1, H5.1, H6.1, U1.2 (VN), SW1.1; no longer U1.5 (VP)
- net RESET: now also SW1.2
- net VBUS: now also U1.5 (VP); no longer U1.2 (VN)
Other:
- moved on the sheet: J2, U4

Commit message: fixed incorrect schematic symbol for mosfet
Parts:
- Q1: value Q_PMOS_DSG -> Q_PMOS_GSD; symbol Device:Q_PMOS_DSG -> Device:Q_PMOS_GSD
Connections:
- net +BATT: now also Q1.3 (D); no longer Q1.1 (D)
- net VBUS: now also Q1.1 (G); no longer Q1.3 (G)
Changed lines of the file:
@@
 	7575 5350 7675 5350
 $Comp
-L Device:Q_PMOS_DSG Q1
+L Device:Q_PMOS_GSD Q1
 U 1 1 605A8A36
 P 7975 5350
 F 0 "Q1" H 8180 5396 50  0000 L CNN
-F 1 "Q_PMOS_DSG" H 8180 5305 50  0000 L CNN
+F 1 "Q_PMOS_GSD" H 8180 5305 50  0000 L CNN
 F 2 "ul_SI2301CDST1GE3:SI2301CDS-T1-GE3" H 8175 5450 50  0001 C CNN
 F 3 "~" H 7975 5350 50  0001 C CNN
