File: plonck.kicad_pcb (KiCad board)
At the start: 2 copper layers, 228.6 x 78.7 mm, 132 parts, among them J1 Battery_connector, J2 SWD, Q1 USB4085-GF-A_REVA, Q2 Q_PMOS_GSD, SW1 SW_Push, U1 SRV05-4, U2 TP4054-42-SOT25-R, U3 nRF52840_holyiot_18010, U4 XC6206PxxxMR-Regulator_Linear

Commit message: more fixing
Parts:
- removed the Q1 at (69.8, 23.4)
- added J1: USB_C_Receptacle_USB2.0, Connector_USB:USB_C_Receptacle_GCT_USB4085, B.Cu at (66.9, 27.4)
- H1, H2, H3, H4, H5, H6: footprint MountingHole:MountingHole_2.7mm_M2.5_Pad_Via -> MountingHole:MountingHole_2.7mm_M2.5_Pad_TopBottom
- U3: footprint PlanckBT-PCB:nRF52840_holyiot_18010_HS_simple -> holyiot-18010:nRF52840_holyiot_18010_HS_simple
- renumbered J1 to J2, J2 to J3, Q2 to Q1
Routing:
- net D+: track 226.8 -> 227.5 mm

Commit message: updated board revision
Other:
- board text added: "Rev B0"
- board text removed: "Rev A0"
Changed lines of the file:
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@@
     (effects (font (size 0.5 0.5) (thickness 0.125)) (justify mirror))
   )
-  (gr_text "Rev A0" (at 89.2048 97.3582) (layer "B.SilkS")
+  (gr_text "Rev B0" (at 89.2048 97.3582) (layer "B.SilkS")
     (effects (font (size 2 2) (thickness 0.5)) (justify mirror))
   )

Commit message: more more fixing
Parts:
- J3: value SWD -> Conn_01x06; footprint Connector_PinHeader_2.54mm:PinHeader_1x05_P2.54mm_Vertical -> Connector:Tag-Connect_TC2030-IDC-NL_2x03_P1.27mm_Vertical
- moved J3 2.74 mm to (256.5, 60.5)
- renumbered R2 to R1, R1 to R2
Connections:
- J3 pad 1: GND -> +3V3
- J3 pad 3: SWCLK -> RESET
- J3 pad 4: RESET -> SWCLK
- J3 pad 5: +3V3 -> GND
Routing:
- net +3V3: track 118.2 -> 109.2 mm
- net SWCLK: track 43.8 -> 49.8 mm
- net GND: track 54.1 -> 52.8 mm
- net SWDIO: track 47.1 -> 46.6 mm, vias 1 -> 2
Other:
- board text removed: "+3.3v"
- board text removed: "GND"
- board text removed: "RESET"
- board text removed: "SWCLK"
- board text removed: "SWDIO"
