File: plonck.kicad_sch (KiCad schematic)
At the start: 132 parts, among them J1 Battery_connector, J2 SWD, Q1 USB4085-GF-A_REVA, Q2 Q_PMOS_GSD, SW1 SW_Push, U1 SRV05-4, U2 TP4054-42-SOT25-R, U3 nRF52840_holyiot_18010, U4 XC6206PxxxMR-Regulator_Linear

Commit message: more fixing
Parts:
- removed Q1: USB4085-GF-A_REVA, USB4085-GF-A:GCT_USB4085-GF-A_REVA, symbol USB4085-GF-A_REVA:USB4085-GF-A_REVA
- added J1: USB_C_Receptacle_USB2.0, Connector_USB:USB_C_Receptacle_GCT_USB4085, symbol Connector:USB_C_Receptacle_USB2.0
- H1, H2, H3, H4, H5, H6: footprint MountingHole:MountingHole_2.7mm_M2.5_Pad_Via -> MountingHole:MountingHole_2.7mm_M2.5_Pad_TopBottom
- U3: footprint PlanckBT-PCB:nRF52840_holyiot_18010_HS_simple -> holyiot-18010:nRF52840_holyiot_18010_HS_simple
- renumbered J1 to J2, J2 to J3, Q2 to Q1
Connections:
- net D+: now also J1.A6 (D+), J1.B6 (D+)
- net D-: now also J1.A7 (D-), J1.B7 (D-)
- net GND: now also J1.A1 (GND), J1.A12 (GND), J1.B1 (GND), J1.B12 (GND), J1.S1 (SHIELD)
- net at F1.2: now also J1.A4 (VBUS), J1.A9 (VBUS), J1.B4 (VBUS), J1.B9 (VBUS)
- net at R2.2: now also J1.A5 (CC1)
- net at R1.2: now also J1.B5 (CC2)
Other:
- moved on the sheet: F1, R1, R2

Commit message: more more fixing
Parts:
- removed J3: SWD, Connector_PinHeader_2.54mm:PinHeader_1x05_P2.54mm_Vertical, symbol plonck-rescue:SWD-Connector_Generic
- added J3: Conn_01x06, Connector:Tag-Connect_TC2030-IDC-NL_2x03_P1.27mm_Vertical, symbol Connector_Generic:Conn_01x06
- renumbered R2 to R1, R1 to R2
Connections:
- net +3V3: now also J3.1 (Pin_1)
- net GND: now also J3.5 (Pin_5)
- net RESET: now also J3.3 (Pin_3)
- net SWCLK: now also J3.4 (Pin_4)
- net SWDIO: now also J3.2 (Pin_2)
- no-connect marks 13 -> 14
Changed lines of the file:
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@@
   (junction (at 248.285 90.805) (diameter 0.9144) (color 0 0 0 0))
   (junction (at 253.365 135.89) (diameter 0.9144) (color 0 0 0 0))
+  (no_connect (at 71.12 187.96))
   (no_connect (at 125.095 131.445))
   (no_connect (at 125.095 133.985))
@@
     (stroke (width 0) (type dash) (color 0 0 0 0))
   )
-  (polyline (pts (xy 60.325 169.545) (xy 60.325 189.23))
+  (polyline (pts (xy 60.325 169.3418) (xy 60.325 169.4434))
     (stroke (width 0) (type dash) (color 0 0 0 0))
   )
-  (polyline (pts (xy 60.325 189.23) (xy 84.455 189.23))
+  (polyline (pts (xy 60.325 169.5958) (xy 60.325 189.6364))
+    (stroke (width 0) (type dash) (color 0 0 0 0))
+  )
+  (polyline (pts (xy 60.325 189.6364) (xy 81.8896 189.6364))
     (stroke (width 0) (type dash) (color 0 0 0 0))
   )
@@
     (stroke (width 0) (type dash) (color 0 0 0 0))
   )
-  (polyline (pts (xy 84.455 166.37) (xy 84.455 140.335))
+  (polyline (pts (xy 81.8896 169.4434) (xy 60.325 169.4434))
     (stroke (width 0) (type dash) (color 0 0 0 0))
   )
-  (polyline (pts (xy 84.455 169.545) (xy 60.325 169.545))
+  (polyline (pts (xy 81.8896 189.6364) (xy 81.8896 169.4434))
     (stroke (width 0) (type dash) (color 0 0 0 0))
   )
-  (polyline (pts (xy 84.455 189.23) (xy 84.455 169.545))
+  (polyline (pts (xy 84.455 166.37) (xy 84.455 140.335))
     (stroke (width 0) (type dash) (color 0 0 0 0))
   )
@@
     )
   )
-  (global_label "SWDIO" (shape input) (at 71.755 179.07 180) (fields_autoplaced)
+  (global_label "SWDIO" (shape input) (at 71.12 177.8 180) (fields_autoplaced)
     (effects (font (size 1.27 1.27)) (justify right))
-    (property "Intersheet References" "${INTERSHEET_REFS}" (id 0) (at 0 0 0)
+    (property "Intersheet References" "${INTERSHEET_REFS}" (id 0) (at -0.635 -1.27 0)
       (effects (font (size 1.27 1.27)) hide)
     )
   )
-  (global_label "SWCLK" (shape input) (at 71.755 181.61 180) (fields_autoplaced)
+  (global_label "RESET" (shape input) (at 71.12 180.34 180) (fields_autoplaced)
     (effects (font (size 1.27 1.27)) (justify right))
-    (property "Intersheet References" "${INTERSHEET_REFS}" (id 0) (at 0 0 0)
+    (property "Intersheet References" "${INTERSHEET_REFS}" (id 0) (at -0.635 -3.81 0)
       (effects (font (size 1.27 1.27)) hide)
     )
   )
-  (global_label "RESET" (shape input) (at 71.755 184.15 180) (fields_autoplaced)
+  (global_label "SWCLK" (shape input) (at 71.12 182.88 180) (fields_autoplaced)
     (effects (font (size 1.27 1.27)) (justify right))
-    (property "Intersheet References" "${INTERSHEET_REFS}" (id 0) (at 0 0 0)
+    (property "Intersheet References" "${INTERSHEET_REFS}" (id 0) (at -0.635 1.27 0)
       (effects (font (size 1.27 1.27)) hide)
     )
@@
     )
   )
-  (symbol (lib_id "power:+3.3V") (at 71.755 186.69 90) (unit 1)
+  (symbol (lib_id "power:+3.3V") (at 71.12 175.26 90) (unit 1)
     (in_bom yes) (on_board yes)
-    (property "Reference" "#PWR037" (id 0) (at 75.565 186.69 0)
+    (property "Reference" "#PWR034" (id 0) (at 74.93 175.26 0)
       (effects (font (size 1.27 1.27)) hide)
     )
-    (property "Value" "+3.3V" (id 1) (at 68.5038 186.309 90)
+    (property "Value" "+3.3V" (id 1) (at 67.8688 174.879 90)
       (effects (font (size 1.27 1.27)) (justify left))
     )
-    (property "Footprint" "" (id 2) (at 71.755 186.69 0)
+    (property "Footprint" "" (id 2) (at 71.12 175.26 0)
       (effects (font (size 1.27 1.27)) hide)
     )
-    (property "Datasheet" "" (id 3) (at 71.755 186.69 0)
+    (property "Datasheet" "" (id 3) (at 71.12 175.26 0)
       (effects (font (size 1.27 1.27)) hide)
     )
@@
     (pin "1")
   )
-  (symbol (lib_id "power:GND") (at 71.755 176.53 270) (unit 1)
+  (symbol (lib_id "power:GND") (at 71.12 185.42 270) (unit 1)
     (in_bom yes) (on_board yes)
-    (property "Reference" "#PWR034" (id 0) (at 65.405 176.53 0)
+    (property "Reference" "#PWR037" (id 0) (at 64.77 185.42 0)
       (effects (font (size 1.27 1.27)) hide)
     )
-    (property "Value" "GND" (id 1) (at 68.5038 176.657 90)
+    (property "Value" "GND" (id 1) (at 67.8688 185.547 90)
       (effects (font (size 1.27 1.27)) (justify right))
     )
-    (property "Footprint" "" (id 2) (at 71.755 176.53 0)
+    (property "Footprint" "" (id 2) (at 71.12 185.42 0)
       (effects (font (size 1.27 1.27)) hide)
     )
-    (property "Datasheet" "" (id 3) (at 71.755 176.53 0)
+    (property "Datasheet" "" (id 3) (at 71.12 185.42 0)
       (effects (font (size 1.27 1.27)) hide)
     )
@@
   (symbol (lib_id "Device:R_Small") (at 212.09 30.48 270) (unit 1)
     (in_bom yes) (on_board yes)
-    (property "Reference" "R2" (id 0) (at 212.09 30.48 90))
+    (property "Reference" "R1" (id 0) (at 212.09 30.48 90))
     (property "Value" "5.1k" (id 1) (at 212.09 28.575 90))
     (property "Footprint" "Resistor_SMD:R_0603_1608Metric" (id 2) (at 212.09 30.48 0)
@@
   (symbol (lib_id "Device:R_Small") (at 212.09 33.02 270) (unit 1)
     (in_bom yes) (on_board yes)
-    (property "Reference" "R1" (id 0) (at 212.09 33.02 90))
+    (property "Reference" "R2" (id 0) (at 212.09 33.02 90))
     (property "Value" "5.1k" (id 1) (at 212.09 34.925 90))
     (property "Footprint" "Resistor_SMD:R_0603_1608Metric" (id 2) (at 212.09 33.02 0)
@@
     (pin "2")
   )
-  (symbol (lib_id "plonck-rescue:SWD-Connector_Generic") (at 75.565 171.45 0) (unit 1)
+  (symbol (lib_id "plonck-rescue:Battery_connector-Connector_Generic") (at 200.025 87.63 0) (unit 1)
     (in_bom yes) (on_board yes)
-    (property "Reference" "J3" (id 0) (at 74.295 171.45 0)
+    (property "Reference" "J2" (id 0) (at 200.025 88.265 0)
       (effects (font (size 1.27 1.27)) (justify left))
     )
-    (property "Value" "SWD" (id 1) (at 74.295 173.355 0)
+    (property "Value" "Battery_connector" (id 1) (at 200.025 90.17 0)
       (effects (font (size 1.27 1.27)) (justify left))
     )
-    (property "Footprint" "Connector_PinHeader_2.54mm:PinHeader_1x05_P2.54mm_Vertical" (id 2) (at 75.565 171.45 0)
+    (property "Footprint" "SM02B-SRSS-TB_LF__SN_:SM02B-SRSS-TB(LF)(SN)" (id 2) (at 200.025 87.63 0)
+      (effects (font (size 1.27 1.27)) hide)
+    )
+    (property "Datasheet" "" (id 3) (at 200.025 87.63 0)
       (effects (font (size 1.27 1.27)) hide)
     )
-    (property "Datasheet" "" (id 3) (at 75.565 171.45 0)
+    (property "LCSC" "" (id 4) (at 200.025 87.63 0)
       (effects (font (size 1.27 1.27)) hide)
     )
@@
     (pin "3")
     (pin "4")
-    (pin "5")
   )
-  (symbol (lib_id "plonck-rescue:Battery_connector-Connector_Generic") (at 200.025 87.63 0) (unit 1)
+  (symbol (lib_id "Connector_Generic:Conn_01x06") (at 76.2 180.34 0) (unit 1)
     (in_bom yes) (on_board yes)
-    (property "Reference" "J2" (id 0) (at 200.025 88.265 0)
+    (property "Reference" "J3" (id 0) (at 73.66 170.8149 0)
       (effects (font (size 1.27 1.27)) (justify left))
     )
-    (property "Value" "Battery_connector" (id 1) (at 200.025 90.17 0)
+    (property "Value" "Conn_01x06" (id 1) (at 69.85 172.0849 0)
       (effects (font (size 1.27 1.27)) (justify left))
     )
-    (property "Footprint" "SM02B-SRSS-TB_LF__SN_:SM02B-SRSS-TB(LF)(SN)" (id 2) (at 200.025 87.63 0)
+    (property "Footprint" "Connector:Tag-Connect_TC2030-IDC-NL_2x03_P1.27mm_Vertical" (id 2) (at 76.2 180.34 0)
       (effects (font (size 1.27 1.27)) hide)
     )
-    (property "Datasheet" "" (id 3) (at 200.025 87.63 0)
-      (effects (font (size 1.27 1.27)) hide)
-    )
-    (property "LCSC" "" (id 4) (at 200.025 87.63 0)
+    (property "Datasheet" "~" (id 3) (at 76.2 180.34 0)
       (effects (font (size 1.27 1.27)) hide)
     )
@@
     (pin "3")
     (pin "4")
+    (pin "5")
+    (pin "6")
   )
   (symbol (lib_id "Device:Q_PMOS_GSD") (at 202.565 135.89 0) (unit 1)
@@
       (reference "#PWR033") (unit 1) (value "+BATT") (footprint "")
     )
-    (path "/00000000-0000-0000-0000-0000607763ae"
-      (reference "#PWR034") (unit 1) (value "GND") (footprint "")
+    (path "/00000000-0000-0000-0000-0000607779fe"
+      (reference "#PWR034") (unit 1) (value "+3.3V") (footprint "")
     )
     (path "/00000000-0000-0000-0000-000060bb02f8"
@@
       (reference "#PWR036") (unit 1) (value "GND") (footprint "")
     )
-    (path "/00000000-0000-0000-0000-0000607779fe"
-      (reference "#PWR037") (unit 1) (value "+3.3V") (footprint "")
+    (path "/00000000-0000-0000-0000-0000607763ae"
+      (reference "#PWR037") (unit 1) (value "GND") (footprint "")
     )
     (path "/00000000-0000-0000-0000-000060625507"
@@
       (reference "J2") (unit 1) (value "Battery_connector") (footprint "SM02B-SRSS-TB_LF__SN_:SM02B-SRSS-TB(LF)(SN)")
     )
-    (path "/00000000-0000-0000-0000-000060775440"
-      (reference "J3") (unit 1) (value "SWD") (footprint "Connector_PinHeader_2.54mm:PinHeader_1x05_P2.54mm_Vertical")
+    (path "/44b4065f-3c05-4e3c-b29a-6a1e2cf5e69c"
+      (reference "J3") (unit 1) (value "Conn_01x06") (footprint "Connector:Tag-Connect_TC2030-IDC-NL_2x03_P1.27mm_Vertical")
     )
     (path "/00000000-0000-0000-0000-0000604e9665"
@@
       (reference "Q1") (unit 1) (value "Q_PMOS_GSD") (footprint "ul_SI2301CDST1GE3:SI2301CDS-T1-GE3")
     )
-    (path "/00000000-0000-0000-0000-0000606709da"
+    (path "/00000000-0000-0000-0000-000060672a19"
       (reference "R1") (unit 1) (value "5.1k") (footprint "Resistor_SMD:R_0603_1608Metric")
     )
-    (path "/00000000-0000-0000-0000-000060672a19"
+    (path "/00000000-0000-0000-0000-0000606709da"
       (reference "R2") (unit 1) (value "5.1k") (footprint "Resistor_SMD:R_0603_1608Metric")
     )
